File: pcb/Robot-Controller_v11.sch (EAGLE design)
At the start: 54 parts, among them IC1 FT232RQ, IC2 LDO-TS1117-5V, IC3 DRV8838, IC4 DRV8838, IC5 DRV8838, IC6 DRV8838, J2 USB10103594-0001LF, M1 1751248, M2 1751248, M3 1751248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

Commit message: cleaned up schematics and layout
Other:
- note removed: "www.watterott.com"
Changed lines of the file:
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@@
 <setting verticaltext="up"/>
 </settings>
-<grid distance="0.1" unitdist="inch" unit="inch" style="lines" multiple="1" display="no" altdistance="0.01" altunitdist="inch" altunit="inch"/>
+<grid distance="0.05" unitdist="inch" unit="inch" style="lines" multiple="1" display="yes" altdistance="0.025" altunitdist="inch" altunit="inch"/>
 <layers>
 <layer number="1" name="Top" color="4" fill="1" visible="no" active="no"/>
@@
 <part name="IC5" library="we-chip" deviceset="DRV8837" device="" value="DRV8838"/>
 <part name="IC6" library="we-chip" deviceset="DRV8837" device="" value="DRV8838"/>
-<part name="FRAME1" library="frames" deviceset="A4L-LOC" device=""/>
 <part name="ARDUINO" library="wattuino" deviceset="WATTUINO_PRO_MINI" device="ADV1.0" technology="5" value="WATTUINO_PRO_MINI"/>
 <part name="T1" library="we-transistor" deviceset="MOSFET_N-CHN" device="-IRLML2502"/>
@@
 <part name="F1" library="we-rcl" deviceset="RESISTOR" device="-R0805" value="0.5A"/>
 <part name="GND18" library="supply1" deviceset="GND" device=""/>
+<part name="FRAME1" library="we-symbol" deviceset="FRAME-A4L" device=""/>
 </parts>
 <sheets>
@@
 <wire x1="123.19" y1="148.59" x2="123.19" y2="149.86" width="1.016" layer="94"/>
 <wire x1="27.94" y1="86.36" x2="27.94" y2="92.71" width="0.1524" layer="94"/>
-<text x="213.36" y="5.08" size="2.54" layer="94" font="vector" align="bottom-right">www.watterott.com</text>
-<text x="161.29" y="31.75" size="1.27" layer="95">Released under the Creative Commons Attribution Share-Alike License</text>
-<text x="161.29" y="29.21" size="1.27" layer="95">http://creativecommons.org/licenses/by-sa/4.0/</text>
-<text x="161.29" y="25.4" size="1.27" layer="95">Designed by Stephan Watterott (Watterott electronic)</text>
+<text x="162.56" y="21.59" size="1.27" layer="95">Released under the Creative Commons Attribution Share-Alike License</text>
+<text x="162.56" y="19.05" size="1.27" layer="95">http://creativecommons.org/licenses/by-sa/4.0/</text>
+<text x="162.56" y="15.24" size="1.27" layer="95">Designed by Stephan Watterott (Watterott electronic)</text>
 </plain>
 <instances>
@@
 <instance part="IC5" gate="IC$1" x="205.74" y="87.63" rot="MR0"/>
 <instance part="IC6" gate="IC$1" x="205.74" y="55.88" rot="MR0"/>
-<instance part="FRAME1" gate="G$1" x="0" y="0"/>
 <instance part="ARDUINO" gate="WATTUINO" x="53.34" y="146.05"/>
 <instance part="T1" gate="T" x="119.38" y="22.86"/>
@@
 <instance part="I2C" gate="J" x="146.05" y="158.75" rot="R180"/>
 <instance part="D3" gate="G$1" x="119.38" y="30.48" rot="R90"/>
-<instance part="LOGO2" gate="G$1" x="193.04" y="19.05"/>
-<instance part="X1" gate="X" x="166.37" y="19.05"/>
-<instance part="X2" gate="X" x="173.99" y="19.05"/>
-<instance part="LOGO3" gate="G$1" x="207.01" y="19.05"/>
+<instance part="LOGO2" gate="G$1" x="198.12" y="7.62"/>
+<instance part="X1" gate="X" x="165.1" y="7.62"/>
+<instance part="X2" gate="X" x="170.18" y="7.62"/>
+<instance part="LOGO3" gate="G$1" x="208.28" y="7.62"/>
 <instance part="POWER" gate="-1" x="29.21" y="22.86" rot="R180"/>
 <instance part="POWER" gate="-2" x="29.21" y="7.62" rot="R180"/>
@@
 <instance part="F1" gate="R" x="27.94" y="90.17" rot="R90"/>
 <instance part="GND18" gate="1" x="135.89" y="46.99" rot="MR0"/>
+<instance part="FRAME1" gate="G$1" x="0" y="0"/>
 </instances>
 <busses>
